File: _Safety System (SS)/A6SS-4/A6SS-4.brd (EAGLE design)
At the start: 66 x 39.4 mm, 117 parts, among them J1 M2M1X2, J2 M2M1X2, Q1 MMBT4403LT3G, Q2 MMBT4403LT3G, U1 PIC18F45K22, U10 MCP6541RT-E/OT, U11 MCP6541RT-E/OT, U12 SN74LVC1G132DBVR, U13 MAX6817EUT+T, U14 MAX823TEUK+T_3.08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

Commit message: SS updates and fixes
Parts:
- moved U$1 9.09 mm to (51.5, 35.1)
Other:
- board text added: "CF"
- board text added: "LR"
