File: _Battery Management/HV/Current sense-done/Current.brd (EAGLE design)
At the start: 114.4 x 32.9 mm, 71 parts, among them J1 M80022232081-2, U1 ADS1015, U10 HV7802, U13 HV7802, U15 HV7802, U16 M5_0.2_ISO, U17 HV7802, U19 HV7802, U2 LR8, U21 M5_0.2_ISO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

Commit message: Current sense updates
Parts:
- added GND, IGND, ISCL, ISDA, SCL, SDA: TPSMD, FSAE Electric:0603
Connections:
- net GND: now also GND.1, GND.2
- net N$7: now also SDA.1, SDA.2
- net N$71: now also ISCL.1, ISCL.2
- net N$72: now also ISDA.1, ISDA.2
- net N$8: now also SCL.1, SCL.2
- net V-: now also IGND.1, IGND.2
Routing:
- net N$8: track 10.4 -> 30.6 mm
- net N$7: track 11.5 -> 31.1 mm
- net N$72: track 105.0 -> 106.0 mm
- net N$71: track 92.5 -> 93.0 mm
- net V-: vias 21 -> 22
