File: _Charger_Done/PCB/Charger_PCB.brd (EAGLE design)
At the start: 67.8 x 86.9 mm, 81 parts, among them J1 M4_1X4_LOCK, J2 M2X5_IDC, K5 OJ-SS-124LMH2, K6 OJ-SS-124LMH2, K7 OJ-SS-124LMH2, K8 OJ-SS-124LMH2, Q1 NUD3160LT1G, Q2 NUD3160LT1G, Q3 NUD3160LT1G, Q4 BSS123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

Commit message: Working on BMM
Parts:
- moved C5 4.51 mm to (8.28, -24.7), turned to 90 degrees
Connections:
- removed net N$41: U11.1, U4.3
- new net N$30: U11.1, U4.2
- net GPIO: now also U8.20
- net N$39: now also U4.3; no longer U4.2
Routing:
- net N$30: track 0.00 -> 6.24 mm
- net N$41: track 3.52 -> 0.00 mm
- net +5V: track 264.6 -> 267.7 mm
- net USBTX: track 9.61 -> 8.93 mm
